Commit message: new cassie model (achilles rods)
addition of achilles rods + reading inertia from file

File: mocca_envs/data/cassie/urdf/cassie_collide.urdf (robot description, URDF)
Before this commit: robot cassie, 18 links, 17 joints
Links:
- added link left_achilles_rod, mass 0.1567; visual mesh filename=../meshes/achilles-rod.stl scale=1 1 1
- added link left_achilles_rod_y, mass 0
- added link right_achilles_rod, mass 0.1567; visual mesh filename=../meshes/achilles-rod.stl scale=1 1 1
- added link right_achilles_rod_y, mass 0
Joints:
- added joint fixed_left_achilles_rod_joint_y: type continuous, parent left_achilles_rod_y, child left_achilles_rod, origin xyz=0 0 0 rpy=0 0 0, axis 0 1 0
- added joint fixed_left_achilles_rod_joint_z: type continuous, parent left_thigh, child left_achilles_rod_y, origin xyz=0 0 0.045 rpy=0 0 0, axis 0 0 1
- added joint fixed_right_achilles_rod_joint_y: type continuous, parent right_achilles_rod_y, child right_achilles_rod, origin xyz=0 0 0 rpy=0 0 0, axis 0 1 0
- added joint fixed_right_achilles_rod_joint_z: type continuous, parent right_thigh, child right_achilles_rod_y, origin xyz=0 0 -0.045 rpy=0 0 0, axis 0 0 1
- joint knee_to_shin_left: limit lower=-0.349 upper=0.349 effort=0 velocity=100 -> lower=-0.0349 upper=0.0349 effort=0 velocity=100
- joint knee_to_shin_right: limit lower=-0.349 upper=0.349 effort=0 velocity=100 -> lower=-0.0349 upper=0.0349 effort=0 velocity=100

File: mocca_envs/data/cassie/urdf/cassie_collide_2d.urdf (robot description, URDF)
Before this commit: robot cassie, 20 links, 19 joints
Links:
- added link left_achilles_rod, mass 0.1567; visual mesh filename=../meshes/achilles-rod.stl scale=1 1 1
- added link left_achilles_rod_y, mass 0
- added link right_achilles_rod, mass 0.1567; visual mesh filename=../meshes/achilles-rod.stl scale=1 1 1
- added link right_achilles_rod_y, mass 0
Joints:
- added joint fixed_left_achilles_rod_joint_y: type continuous, parent left_achilles_rod_y, child left_achilles_rod, origin xyz=0 0 0 rpy=0 0 0, axis 0 1 0
- added joint fixed_left_achilles_rod_joint_z: type continuous, parent left_thigh, child left_achilles_rod_y, origin xyz=0 0 0.045 rpy=0 0 0, axis 0 0 1
- added joint fixed_right_achilles_rod_joint_y: type continuous, parent right_achilles_rod_y, child right_achilles_rod, origin xyz=0 0 0 rpy=0 0 0, axis 0 1 0
- added joint fixed_right_achilles_rod_joint_z: type continuous, parent right_thigh, child right_achilles_rod_y, origin xyz=0 0 -0.045 rpy=0 0 0, axis 0 0 1
- joint knee_to_shin_left: limit lower=-0.349 upper=0.349 effort=0 velocity=100 -> lower=-0.0349 upper=0.0349 effort=0 velocity=100
- joint knee_to_shin_right: limit lower=-0.349 upper=0.349 effort=0 velocity=100 -> lower=-0.0349 upper=0.0349 effort=0 velocity=100

Commit message: reverting to using PD for knee-to-shin springs

File: mocca_envs/data/cassie/urdf/cassie_collide.urdf (robot description, URDF)
Before this commit: robot cassie, 22 links, 21 joints
Joints:
- joint knee_to_shin_left: limit lower=-0.0349 upper=0.0349 effort=0 velocity=100 -> lower=-0.349 upper=0.349 effort=0 velocity=100
- joint knee_to_shin_right: limit lower=-0.0349 upper=0.0349 effort=0 velocity=100 -> lower=-0.349 upper=0.349 effort=0 velocity=100

Commit message: cassie mirror env

File: mocca_envs/data/cassie/urdf/cassie_collide.urdf (robot description, URDF)
Before this commit: robot cassie, 22 links, 21 joints
Joints:
- joint knee_to_shin_left: limit lower=-0.349 upper=0.349 effort=0 velocity=100 -> lower=-0.0349 upper=0.0349 effort=0 velocity=100
- joint knee_to_shin_right: limit lower=-0.349 upper=0.349 effort=0 velocity=100 -> lower=-0.0349 upper=0.0349 effort=0 velocity=100

Commit message: Cassie parameters further tuned + Blue Color

File: mocca_envs/data/cassie/urdf/cassie_collide.urdf (robot description, URDF)
Before this commit: robot cassie, 22 links, 21 joints
Joints:
- joint knee_to_shin_left: limit lower=-0.0349 upper=0.0349 effort=0 velocity=100 -> lower=-0.07 upper=0.07 effort=0 velocity=100
- joint knee_to_shin_right: limit lower=-0.0349 upper=0.0349 effort=0 velocity=100 -> lower=-0.07 upper=0.07 effort=0 velocity=100

File: mocca_envs/data/cassie/urdf/cassie_collide_2d.urdf (robot description, URDF)
Before this commit: robot cassie, 24 links, 23 joints
Joints:
- joint knee_to_shin_left: limit lower=-0.0349 upper=0.0349 effort=0 velocity=100 -> lower=-0.07 upper=0.07 effort=0 velocity=100
- joint knee_to_shin_right: limit lower=-0.0349 upper=0.0349 effort=0 velocity=100 -> lower=-0.07 upper=0.07 effort=0 velocity=100
