Commit message: add mike

File: mocca_envs/data/objects/steps/plank.urdf (robot description, URDF)
Before this commit: robot plank, 2 links, 1 joints
Links:
- link base: geometry collision box size=1 1.5 0.45; visual box size=1 1.5 0.45
- link cover: geometry collision box size=1 1.5 0.05; visual box size=1 1.5 0.05
