Commit message: Fix Laikago model toe collision detection; other env bugfixes

File: mocca_envs/data/robots/laikago/laikago_toes_limits.urdf (robot description, URDF)
Before this commit: robot plane, 17 links, 16 joints
Links:
- link toeFL: geometry collision sphere radius=0.035; visual sphere radius=0.035
- link toeFR: geometry collision sphere radius=0.035; visual sphere radius=0.035
- link toeRL: geometry collision sphere radius=0.035; visual sphere radius=0.035
- link toeRR: geometry collision sphere radius=0.035; visual sphere radius=0.035
Joints:
- joint jtoeFL: origin xyz=0 -0.25 -0.022 -> xyz=0 -0.265 -0.022
- joint jtoeFR: origin xyz=0 -0.25 -0.022 -> xyz=0 -0.265 -0.022
- joint jtoeRL: origin xyz=0 -0.25 -0.022 -> xyz=0 -0.265 -0.022
- joint jtoeRR: origin xyz=0 -0.25 -0.022 -> xyz=0 -0.265 -0.022

Commit message: Increase Laikago torque, add posture penalty, increase size of toes

File: mocca_envs/data/robots/laikago/laikago_toes_limits.urdf (robot description, URDF)
Before this commit: robot plane, 17 links, 16 joints
Links:
- link toeFL: geometry collision sphere radius=0.045; visual sphere radius=0.045
- link toeFR: geometry collision sphere radius=0.045; visual sphere radius=0.045
- link toeRL: geometry collision sphere radius=0.045; visual sphere radius=0.045
- link toeRR: geometry collision sphere radius=0.045; visual sphere radius=0.045
Joints:
- joint jtoeFL: origin xyz=0 -0.265 -0.022 -> xyz=0 -0.27 -0.022
- joint jtoeFR: origin xyz=0 -0.265 -0.022 -> xyz=0 -0.27 -0.022
- joint jtoeRL: origin xyz=0 -0.265 -0.022 -> xyz=0 -0.27 -0.022
- joint jtoeRR: origin xyz=0 -0.265 -0.022 -> xyz=0 -0.27 -0.022

Commit message: Reduce max solver iteration from 20 to 5; change laikago model's default orientation, lower leg length, and toe contact parameters; lots of env changes

File: mocca_envs/data/robots/laikago/laikago_toes_limits.urdf (robot description, URDF)
Before this commit: robot plane, 17 links, 16 joints
Links:
- link FL_lower_leg: geometry collision mesh filename=lower_leg_3.stl scale=0.8 0.8 0.8; visual mesh filename=lower_leg3.obj scale=1 1 1
- link FR_lower_leg: geometry collision mesh filename=lower_leg_3.stl scale=0.8 0.8 0.8; visual mesh filename=lower_leg3.obj scale=1 1 1
- link RL_lower_leg: geometry collision mesh filename=lower_leg_3.stl scale=0.8 0.8 0.8; visual mesh filename=lower_leg3.obj scale=1 1 1
- link RR_lower_leg: geometry collision mesh filename=lower_leg_3.stl scale=0.8 0.8 0.8; visual mesh filename=lower_leg3.obj scale=1 1 1
